Commit message: checks on mac and bugfixes

File: examples/urdf/robot_models/rbot.urdf (robot description, URDF)
Before this commit: robot RBot_description, 2 links, 1 joints
Links:
- added link eef, mass 1; collision sphere radius=0.1; visual sphere radius=0.1
- link link0: mass 1 -> 0.5; geometry collision cylinder length=0.79 radius=0.07; visual cylinder length=1.0 radius=0.07
Joints:
- added joint jfixed: type fixed, parent link0, child eef, origin xyz=0.0 0.0 -1.0 rpy=0 0 0
